File: GlowClockPCB/GlowClockPCB.kicad_sch (KiCad schematic)
At the start: 52 parts, among them J1 LED_OUT_1, J2 LED_OUT_2, J3 LED_OUT_3, J4 LED_OUT_4, J5 POWER_IN, J6 Motor_1_Out, J7 Motor_2_Out, J8 I2C_LCD, J9 ADC_OUT, SW1 BTN_UP, SW2 BTN_LEFT, SW3 BTN_DOWN, SW4 BTN_RIGHT, SW5 BTN_OK, SW6 BTN_BACK, U1 RaspberryPi_Pico_W, U2 Raspberry_Pi_Zero_2_W, U3 DS3231MZ

Commit message: add ability to display images, use pillow to convert images to pixel array of requisite size
Other:
- note added: "SCL"
- note added: "SDA"
Changed lines of the file:
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@@
+		)
+	)
+	(text "SCL"
+		(exclude_from_sim no)
+		(at 204.47 112.522 0)
+		(effects
+			(font
+				(size 1.27 1.27)
+			)
+		)
+	)
+	(text "SDA"
+		(exclude_from_sim no)
+		(at 204.47 115.062 0)
+		(effects
+			(font
+				(size 1.27 1.27)
+			)
 		)
 	)
